File: output/pcbs/main.kicad_pcb (KiCad board)
At the start: 2 copper layers, 154.4 x 118.3 mm, 64 parts

Commit message: routing for V1.0 with logo and text
Parts:
- added G***: LOGO, falkbrand:logo2, F.Cu at (181.9, 136.8)
- added G***: LOGO, falkbrand:logo2_B, F.Cu at (179.8, 134.0)
- moved D15 0.29 mm to (177.5, 100.2)
- moved S14 0.29 mm to (179.6, 112.0)
- moved S12 0.29 mm to (157.1, 88.0)
- moved S7 0.29 mm to (140.2, 127.4)
- moved D28 0.29 mm to (191.3, 146.4)
- moved D9 0.29 mm to (167.5, 147.1)
- moved D18 0.29 mm to (202.0, 122.9)
- moved S22 0.29 mm to (220.0, 116.8)
- moved D1 0.29 mm to (137.6, 173.0)
- moved D13 0.29 mm to (183.8, 135.6)
- moved D16 0.29 mm to (174.4, 82.4)
- moved D19 0.29 mm to (201.9, 104.9)
- moved D2 0.29 mm to (131.5, 156.1)
- moved D21 0.29 mm to (220.2, 140.8)
- moved D22 0.29 mm to (220.0, 122.8)
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Routing:
- net RST: track 6.22 -> 57.2 mm, vias 0 -> 2
- net GND: track 63.4 -> 80.0 mm
- net ring_top: track 30.3 -> 32.4 mm
- net P20: track 220.1 -> 222.3 mm
- net P4: track 192.3 -> 190.4 mm
- net thumb_home: track 32.2 -> 33.8 mm
Other:
- board text added: "elfalko/FOCK V1.0"

Commit message: V2 production ready
Parts:
- removed B2: , E73:SW_TACT_ALPS_SKQGABE010
- removed G***: LOGO, falkbrand:logo2
- removed G***: LOGO, falkbrand:logo2_B
- removed PAD1, PAD2: , SMDPad
- removed the REF** at (256.2, 143.4)
- added ?: +, Text, F.Cu at (127.7, 27.7)
- added ?: , SMDPad, F.Cu at (130.5, 14.0)
- added ?: , SMDPad, F.Cu at (129.5, 16.8)
- added ?: +, Text, B.Cu at (127.7, 27.7)
- added ?: -, Text, F.Cu at (129.9, 21.4)
- added ?: -, Text, B.Cu at (129.9, 21.4)
- added ?: LOGO, LOGO, F.Cu at (69.1, -19.1)
- added ?: LOGO, LOGO, B.Cu at (69.1, -19.1)
- added ?: elfalko/FOCK V2.0, Text, F.Cu at (146.7, -3.59)
- added ?: elfalko/FOCK V2.0, Text, B.Cu at (146.7, -3.59)
- added ?: JLCJLCJLCJLC, Text, F.Cu at (124.0, -5.28)
- added J1: , solderjumper, F.Cu at (129.2, 26.8)
- added J2: , solderjumper, F.Cu at (127.3, 26.1)
- added J3: , solderjumper, F.Cu at (130.5, 23.0)
- added J4: , solderjumper, F.Cu at (128.6, 22.4)
- added JST1: , JST_PH_S2B-PH-K_02x2.00mm_Angled, F.Cu at (128.9, 24.6)
- added PAD5: , SMDPad, F.Cu at (108.7, 12.4)
- added PAD6: , SMDPad, F.Cu at (108.7, 11.8)
- added REF**: VIA-0.3mm, VIA-0.3mm, F.Cu at (23.5, -8.00)
- added REF**: VIA-0.3mm, VIA-0.3mm, F.Cu at (34.2, -3.75)
- added REF**: VIA-0.3mm, VIA-0.3mm, F.Cu at (41.5, -26.0)
- added REF**: VIA-0.3mm, VIA-0.3mm, F.Cu at (34.2, -21.8)
- added REF**: VIA-0.3mm, VIA-0.3mm, F.Cu at (41.5, -44.0)
- added REF**: VIA-0.3mm, VIA-0.3mm, F.Cu at (34.2, -39.8)
- added REF**: VIA-0.3mm, VIA-0.3mm, F.Cu at (41.5, -62.0)
- added REF**: VIA-0.3mm, VIA-0.3mm, F.Cu at (34.2, -57.8)
- added REF**: VIA-0.3mm, VIA-0.3mm, F.Cu at (62.8, -20.9)
- added REF**: VIA-0.3mm, VIA-0.3mm, F.Cu at (54.9, -18.0)
- added REF**: VIA-0.3mm, VIA-0.3mm, F.Cu at (65.9, -38.6)
- added REF**: VIA-0.3mm, VIA-0.3mm, F.Cu at (16.2, -3.75)
- added REF**: VIA-0.3mm, VIA-0.3mm, F.Cu at (58.1, -35.7)
- added REF**: VIA-0.3mm, VIA-0.3mm, F.Cu at (69.1, -56.4)
- added REF**: VIA-0.3mm, VIA-0.3mm, F.Cu at (61.2, -53.4)
- added REF**: VIA-0.3mm, VIA-0.3mm, F.Cu at (72.2, -74.1)
- added REF**: VIA-0.3mm, VIA-0.3mm, F.Cu at (64.3, -71.2)
- added REF**: VIA-0.3mm, VIA-0.3mm, F.Cu at (82.0, -26.2)
- added REF**: VIA-0.3mm, VIA-0.3mm, F.Cu at (74.1, -23.2)
- added REF**: VIA-0.3mm, VIA-0.3mm, F.Cu at (85.1, -43.9)
- added REF**: VIA-0.3mm, VIA-0.3mm, F.Cu at (77.3, -41.0)
- added REF**: VIA-0.3mm, VIA-0.3mm, F.Cu at (88.3, -61.6)
- added REF**: VIA-0.3mm, VIA-0.3mm, F.Cu at (23.5, -26.0)
- added REF**: VIA-0.3mm, VIA-0.3mm, F.Cu at (80.4, -58.7)
- added REF**: VIA-0.3mm, VIA-0.3mm, F.Cu at (91.4, -79.3)
- added REF**: VIA-0.3mm, VIA-0.3mm, F.Cu at (83.5, -76.4)
- added REF**: VIA-0.3mm, VIA-0.3mm, F.Cu at (99.5, -13.4)
- added REF**: VIA-0.3mm, VIA-0.3mm, F.Cu at (91.3, -11.8)
- added REF**: VIA-0.3mm, VIA-0.3mm, F.Cu at (105.5, -30.4)
- added REF**: VIA-0.3mm, VIA-0.3mm, F.Cu at (97.3, -28.8)
- added REF**: VIA-0.3mm, VIA-0.3mm, F.Cu at (111.5, -47.4)
- added REF**: VIA-0.3mm, VIA-0.3mm, F.Cu at (103.3, -45.8)
- added REF**: VIA-0.3mm, VIA-0.3mm, F.Cu at (117.5, -64.3)
- added REF**: VIA-0.3mm, VIA-0.3mm, F.Cu at (16.2, -21.8)
- added REF**: VIA-0.3mm, VIA-0.3mm, F.Cu at (109.3, -62.7)
- added REF**: VIA-0.3mm, VIA-0.3mm, F.Cu at (116.5, -7.41)
- added REF**: VIA-0.3mm, VIA-0.3mm, F.Cu at (108.2, -5.82)
- added REF**: VIA-0.3mm, VIA-0.3mm, F.Cu at (122.5, -24.4)
- added REF**: VIA-0.3mm, VIA-0.3mm, F.Cu at (114.2, -22.8)
- added REF**: VIA-0.3mm, VIA-0.3mm, F.Cu at (128.5, -41.3)
- added REF**: VIA-0.3mm, VIA-0.3mm, F.Cu at (120.2, -39.8)
- added REF**: VIA-0.3mm, VIA-0.3mm, F.Cu at (134.5, -58.3)
- added REF**: VIA-0.3mm, VIA-0.3mm, F.Cu at (126.2, -56.7)
- added REF**: VIA-0.3mm, VIA-0.3mm, F.Cu at (112.9, 35.4)
- added REF**: VIA-0.3mm, VIA-0.3mm, F.Cu at (23.5, -44.0)
- added REF**: VIA-0.3mm, VIA-0.3mm, F.Cu at (121.3, 35.3)
- added REF**: VIA-0.3mm, VIA-0.3mm, F.Cu at (97.2, 26.6)
- added REF**: VIA-0.3mm, VIA-0.3mm, F.Cu at (105.6, 26.4)
- added REF**: VIA-0.3mm, VIA-0.3mm, F.Cu at (81.6, 17.7)
- added REF**: VIA-0.3mm, VIA-0.3mm, F.Cu at (90.0, 17.6)
- added REF**: VIA-0.3mm, VIA-0.3mm, F.Cu at (65.9, 8.84)
- added REF**: VIA-0.3mm, VIA-0.3mm, F.Cu at (74.3, 8.71)
- added REF**: VIA-0.2mm, VIA-0.2mm, F.Cu at (134.7, 17.1)
- added REF**: VIA-0.2mm, VIA-0.2mm, F.Cu at (135.7, 17.4)
- added REF**: VIA-0.2mm, VIA-0.2mm, F.Cu at (136.6, 17.8)
- added REF**: VIA-0.3mm, VIA-0.3mm, F.Cu at (16.2, -39.8)
- added REF**: VIA-0.2mm, VIA-0.2mm, F.Cu at (137.6, 18.1)
- added REF**: VIA-0.2mm, VIA-0.2mm, F.Cu at (137.8, 19.3)
- added REF**: VIA-0.2mm, VIA-0.2mm, F.Cu at (139.3, 17.3)
- added REF**: VIA-0.2mm, VIA-0.2mm, F.Cu at (135.6, 14.7)
- added REF**: VIA-0.2mm, VIA-0.2mm, F.Cu at (133.9, 19.4)
- added REF**: VIA-0.2mm, VIA-0.2mm, F.Cu at (136.8, 14.4)
- added REF**: VIA-0.2mm, VIA-0.2mm, F.Cu at (134.6, 20.5)
- added REF**: VIA-0.3mm, VIA-0.3mm, F.Cu at (120.3, -7.84)
- added REF**: VIA-0.3mm, VIA-0.3mm, F.Cu at (129.8, 28.9)
- added REF**: VIA-0.3mm, VIA-0.3mm, F.Cu at (132.9, 26.0)
- added REF**: VIA-0.3mm, VIA-0.3mm, F.Cu at (23.5, -62.0)
- added REF**: VIA-0.3mm, VIA-0.3mm, F.Cu at (16.2, -57.8)
- added REF**: VIA-0.3mm, VIA-0.3mm, F.Cu at (41.5, -8.00)
- added T1, T2: , E73:SPDT_C128955, F.Cu at (133.3, 30.9)
- added USB1: , USB-C-12-Pin-MidMount, F.Cu at (140.4, 19.1)
- added USB2: , USB-C-12-Pin-MidMount, B.Cu at (140.4, 19.1)
- moved S1 204.5 mm to (18.0, 0.00), turned to 0 degrees
- moved D1 204.2 mm to (24.8, 2.80), turned to 80 degrees
- moved S2 202.0 mm to (18.0, -18.0), turned to 0 degrees
- moved D2 201.8 mm to (24.8, -15.2), turned to 80 degrees
- moved S3 199.5 mm to (18.0, -36.0), turned to 0 degrees
- moved D3 199.5 mm to (24.8, -33.2), turned to 80 degrees
- moved S5 198.9 mm to (36.0, 0.00), turned to 0 degrees
- moved D5 198.5 mm to (42.8, 2.80), turned to 80 degrees
- moved D4 197.5 mm to (24.8, -51.2), turned to 80 degrees
- moved S4 197.3 mm to (18.0, -54.0), turned to 0 degrees
- moved S6 196.2 mm to (36.0, -18.0), turned to 0 degrees
- moved D6 196.0 mm to (42.8, -15.2), turned to 80 degrees
- moved PAD4 195.8 mm to (108.7, 12.9), turned to 150.5 degrees
- moved S7 193.8 mm to (36.0, -36.0), turned to 0 degrees
- moved PAD3 193.7 mm to (108.7, 13.5), turned to 150.5 degrees
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Connections:
- D1 pad 2: P18 -> outer_bottom
- D10 pad 2: P19 -> ring_home
- D13 pad 1: middle_bottom -> P18
- D13 pad 2: P18 -> middle_bottom
- D17 pad 1: index_bottom -> P18
- D18 pad 2: P19 -> index_home
- D19 pad 1: index_top -> P20
- D20 pad 2: P21 -> index_num
- D21 pad 2: P18 -> inner_bottom
- D25 pad 1: thumb_bottom -> P18
- D25 pad 2: P21 -> thumb_bottom
- D26 pad 1: thumb_home -> P19
- D27 pad 1: thumb_top -> P20
- D28 pad 1: P18 -> P21
- D3 pad 2: P20 -> outer_top
- D4 pad 1: outer_num -> P21
- D7 pad 2: P20 -> pinky_top
- D9 pad 1: ring_bottom -> P18
- PAD3 pad 1: P4 -> P9
- PAD4 pad 1: P3 -> P8
Routing:
- net (no net): track 0.00 -> 3424.5 mm
- net P9: track 276.4 -> 0.00 mm, vias 1 -> 0
- net P8: track 253.4 -> 0.00 mm, vias 4 -> 0
- net P21: track 247.6 -> 0.00 mm, vias 7 -> 0
- net P20: track 222.3 -> 0.00 mm, vias 6 -> 0
- net P7: track 215.6 -> 0.00 mm, vias 2 -> 0
- net P6: track 209.4 -> 0.00 mm, vias 2 -> 0
- net P19: track 197.7 -> 0.00 mm, vias 5 -> 0
- net P4: track 190.4 -> 0.00 mm, vias 3 -> 0
- net P18: track 183.3 -> 0.00 mm
- net P5: track 170.6 -> 0.00 mm, vias 3 -> 0
- net P10: track 147.6 -> 0.00 mm, vias 3 -> 0
- net GND: track 80.0 -> 0.00 mm
- net RST: track 57.2 -> 0.00 mm, vias 2 -> 0
- net RAW: track 54.2 -> 0.00 mm
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Other:
- board size 154.4 x 118.3 mm -> 147 x 131.8 mm
- net class Default added: clearance 0.2, trace_width 0.25, via_dia 0.8, via_drill 0.4
- board text removed: "elfalko/FOCK V1.0"

Commit message: V2 footprint kicad
Parts:
- removed the ? at (127.7, 27.7) (x2)
- removed the ? at (130.5, 14.0)
- removed the ? at (129.5, 16.8)
- removed the ? at (129.9, 21.4) (x2)
- removed the ? at (69.1, -19.1) (x2)
- removed the ? at (146.7, -3.59) (x2)
- removed the ? at (124.0, -5.28)
- removed the REF** at (62.8, -20.9)
- removed the REF** at (54.9, -18.0)
- removed the REF** at (65.9, -38.6)
- removed the REF** at (58.1, -35.7)
- removed the REF** at (69.1, -56.4)
- removed the REF** at (61.2, -53.4)
- removed the REF** at (72.2, -74.1)
- removed the REF** at (64.3, -71.2)
- removed the REF** at (82.0, -26.2)
- removed the REF** at (74.1, -23.2)
- removed the REF** at (85.1, -43.9)
- removed the REF** at (77.3, -41.0)
- removed the REF** at (88.3, -61.6)
- removed the REF** at (80.4, -58.7)
- removed the REF** at (91.4, -79.3)
- removed the REF** at (83.5, -76.4)
- removed the REF** at (99.5, -13.4)
- removed the REF** at (91.3, -11.8)
- removed the REF** at (105.5, -30.4)
- removed the REF** at (97.3, -28.8)
- removed the REF** at (111.5, -47.4)
- removed the REF** at (103.3, -45.8)
- removed the REF** at (117.5, -64.3)
- removed the REF** at (109.3, -62.7)
- removed the REF** at (116.5, -7.41)
- removed the REF** at (108.2, -5.82)
- removed the REF** at (122.5, -24.4)
- removed the REF** at (114.2, -22.8)
- removed the REF** at (128.5, -41.3)
- removed the REF** at (120.2, -39.8)
- removed the REF** at (134.5, -58.3)
- removed the REF** at (126.2, -56.7)
- removed the REF** at (112.9, 35.4)
- removed the REF** at (121.3, 35.3)
- removed the REF** at (97.2, 26.6)
- removed the REF** at (105.6, 26.4)
- removed the REF** at (81.6, 17.7)
- removed the REF** at (90.0, 17.6)
- removed the REF** at (65.9, 8.84)
- removed the REF** at (74.3, 8.71)
- removed the REF** at (134.7, 17.1)
- removed the REF** at (135.7, 17.4)
- removed the REF** at (136.6, 17.8)
- removed the REF** at (137.6, 18.1)
- removed the REF** at (137.8, 19.3)
- removed the REF** at (139.3, 17.3)
- removed the REF** at (135.6, 14.7)
- removed the REF** at (133.9, 19.4)
- removed the REF** at (136.8, 14.4)
- removed the REF** at (134.6, 20.5)
- removed the REF** at (120.3, -7.84)
- removed the REF** at (129.8, 28.9)
- removed the REF** at (132.9, 26.0)
- added ?: , SMDPad, F.Cu at (129.5, 16.8)
- added ?: LOGO, LOGO, B.Cu at (69.1, -19.1)
- added ?: -, Text, B.Cu at (129.9, 21.4)
- added ?: +, Text, F.Cu at (127.7, 27.7)
- added ?: LOGO, LOGO, F.Cu at (69.1, -19.1)
- added ?: JLCJLCJLCJLC, Text, F.Cu at (124.0, -5.28)
- added ?: , SMDPad, F.Cu at (130.5, 14.0)
- added ?: elfalko/FOCK V2.0, Text, F.Cu at (146.7, -3.59)
- added ?: -, Text, F.Cu at (129.9, 21.4)
- added ?: +, Text, B.Cu at (127.7, 27.7)
- added ?: elfalko/FOCK V2.0, Text, B.Cu at (146.7, -3.59)
- added REF**: VIA-0.3mm, VIA-0.3mm, F.Cu at (128.5, -41.3)
- added REF**: VIA-0.3mm, VIA-0.3mm, F.Cu at (82.0, -26.2)
- added REF**: VIA-0.3mm, VIA-0.3mm, F.Cu at (122.5, -24.4)
- added REF**: VIA-0.3mm, VIA-0.3mm, F.Cu at (103.3, -45.8)
- added REF**: VIA-0.3mm, VIA-0.3mm, F.Cu at (72.2, -74.1)
- added REF**: VIA-0.3mm, VIA-0.3mm, F.Cu at (133.9, 19.4)
- added REF**: VIA-0.3mm, VIA-0.3mm, F.Cu at (136.8, 14.4)
- added REF**: VIA-0.3mm, VIA-0.3mm, F.Cu at (105.6, 26.4)
- added REF**: VIA-0.3mm, VIA-0.3mm, F.Cu at (114.2, -22.8)
- added REF**: VIA-0.3mm, VIA-0.3mm, F.Cu at (105.5, -30.4)
- added REF**: VIA-0.3mm, VIA-0.3mm, F.Cu at (109.3, -62.7)
- added REF**: VIA-0.3mm, VIA-0.3mm, F.Cu at (134.5, -58.3)
- added REF**: VIA-0.3mm, VIA-0.3mm, F.Cu at (81.6, 17.7)
- added REF**: VIA-0.3mm, VIA-0.3mm, F.Cu at (132.9, 26.0)
- added REF**: VIA-0.3mm, VIA-0.3mm, F.Cu at (137.6, 18.1)
- added REF**: VIA-0.3mm, VIA-0.3mm, F.Cu at (90.0, 17.6)
- added REF**: VIA-0.3mm, VIA-0.3mm, F.Cu at (97.2, 26.6)
- added REF**: VIA-0.3mm, VIA-0.3mm, F.Cu at (91.3, -11.8)
- added REF**: VIA-0.3mm, VIA-0.3mm, F.Cu at (97.3, -28.8)
- added REF**: VIA-0.3mm, VIA-0.3mm, F.Cu at (58.1, -35.7)
- added REF**: VIA-0.3mm, VIA-0.3mm, F.Cu at (126.2, -56.7)
- added REF**: VIA-0.3mm, VIA-0.3mm, F.Cu at (77.3, -41.0)
- added REF**: VIA-0.3mm, VIA-0.3mm, F.Cu at (117.5, -64.3)
- added REF**: VIA-0.3mm, VIA-0.3mm, F.Cu at (135.6, 14.7)
- added REF**: VIA-0.3mm, VIA-0.3mm, F.Cu at (91.4, -79.3)
- added REF**: VIA-0.3mm, VIA-0.3mm, F.Cu at (69.1, -56.4)
- added REF**: VIA-0.3mm, VIA-0.3mm, F.Cu at (62.8, -20.9)
- added REF**: VIA-0.3mm, VIA-0.3mm, F.Cu at (136.6, 17.8)
- added REF**: VIA-0.3mm, VIA-0.3mm, F.Cu at (83.5, -76.4)
- added REF**: VIA-0.3mm, VIA-0.3mm, F.Cu at (112.9, 35.4)
- added REF**: VIA-0.3mm, VIA-0.3mm, F.Cu at (108.2, -5.82)
- added REF**: VIA-0.3mm, VIA-0.3mm, F.Cu at (61.2, -53.4)
- added REF**: VIA-0.3mm, VIA-0.3mm, F.Cu at (121.3, 35.3)
- added REF**: VIA-0.3mm, VIA-0.3mm, F.Cu at (88.3, -61.6)
- added REF**: VIA-0.3mm, VIA-0.3mm, F.Cu at (80.4, -58.7)
- added REF**: VIA-0.3mm, VIA-0.3mm, F.Cu at (65.9, -38.6)
- added REF**: VIA-0.3mm, VIA-0.3mm, F.Cu at (116.5, -7.41)
- added REF**: VIA-0.3mm, VIA-0.3mm, F.Cu at (120.2, -39.8)
- added REF**: VIA-0.3mm, VIA-0.3mm, F.Cu at (129.8, 28.9)
- added REF**: VIA-0.3mm, VIA-0.3mm, F.Cu at (135.7, 17.4)
- added REF**: VIA-0.3mm, VIA-0.3mm, F.Cu at (139.3, 17.3)
- added REF**: VIA-0.3mm, VIA-0.3mm, F.Cu at (134.6, 20.5)
- added REF**: VIA-0.3mm, VIA-0.3mm, F.Cu at (74.3, 8.71)
- added REF**: VIA-0.3mm, VIA-0.3mm, F.Cu at (120.3, -7.70)
- added REF**: VIA-0.3mm, VIA-0.3mm, F.Cu at (111.5, -47.4)
- added REF**: VIA-0.3mm, VIA-0.3mm, F.Cu at (99.5, -13.4)
- added REF**: VIA-0.3mm, VIA-0.3mm, F.Cu at (137.8, 19.3)
- added REF**: VIA-0.3mm, VIA-0.3mm, F.Cu at (85.1, -43.9)
- added REF**: VIA-0.3mm, VIA-0.3mm, F.Cu at (65.9, 8.84)
- added REF**: VIA-0.3mm, VIA-0.3mm, F.Cu at (54.9, -18.0)
- added REF**: VIA-0.3mm, VIA-0.3mm, F.Cu at (64.3, -71.2)
- added REF**: VIA-0.3mm, VIA-0.3mm, F.Cu at (134.7, 17.1)
- added REF**: VIA-0.3mm, VIA-0.3mm, F.Cu at (74.1, -23.2)
Routing:
- net (no net): track 3424.5 -> 0.00 mm
- net P21: track 0.00 -> 311.8 mm
- net P9: track 0.00 -> 294.6 mm
- net P8: track 0.00 -> 278.7 mm
- net P20: track 0.00 -> 270.1 mm
- net P19: track 0.00 -> 254.2 mm
- net P6: track 0.00 -> 235.3 mm
- net P7: track 0.00 -> 233.2 mm
- net P10: track 0.00 -> 177.6 mm
- net P5: track 0.00 -> 176.0 mm
- net P4: track 0.00 -> 168.2 mm
- net P18: track 0.00 -> 154.7 mm
- net GND: track 0.00 -> 94.3 mm
- net RAW: track 0.00 -> 78.8 mm
- net P3: track 0.00 -> 51.5 mm
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Other:
- net class Default removed
